File: magazine-amp.sch (KiCad schematic (older format))
At the start: 55 parts, among them J1 Input, J2 Output, J3 Output, Q1 МП39Б, Q2 МП39Б, Q3 МП41, Q4 МП42Б, Q5 МП42Б, Q6 П214А, Q7 П214А

Commit message: Finish schematics
Parts:
- C1, C7: footprint (none) -> Capacitor_THT:C_Disc_D4.7mm_W2.5mm_P5.00mm
- C10: value 200n x 15V -> 200u x 15V; footprint (none) -> Capacitor_THT:CP_Radial_D12.5mm_P5.00mm
- C11, C13: value 50n x 6V -> 50u x 6V; footprint (none) -> Capacitor_THT:CP_Radial_D8.0mm_P3.50mm
- C12: value 10n -> 1n; footprint (none) -> Capacitor_THT:C_Disc_D4.7mm_W2.5mm_P5.00mm
- C14: value 10n x 30V -> 1u x 30V; footprint (none) -> Capacitor_THT:CP_Radial_D8.0mm_P3.50mm
- C2: value 5n x 6V -> 5u x 6V; footprint (none) -> Capacitor_THT:CP_Radial_D4.0mm_P2.00mm
- C3: value 10n x 10V -> 10u x 10V; footprint (none) -> Capacitor_THT:CP_Radial_D7.5mm_P2.50mm
- C4: value 22n x 30V -> 22u x 30V; footprint (none) -> Capacitor_THT:CP_Radial_D10.0mm_P5.00mm
- C5: footprint (none) -> Capacitor_THT:C_Disc_D10.0mm_W2.5mm_P5.00mm
- C6: footprint (none) -> Capacitor_THT:C_Rect_L11.0mm_W3.4mm_P10.00mm_MKT
- C8: value 10 ??? -> 100n; footprint (none) -> Capacitor_THT:C_Rect_L11.0mm_W3.4mm_P10.00mm_MKT
- C9: footprint (none) -> Capacitor_THT:CP_Radial_D7.5mm_P2.50mm
- J1, J2, RV1, RV2, RV3, RV4, RV5: footprint (none) -> Connector_PinSocket_2.54mm:PinSocket_1x02_P2.54mm_Vertical
- J3: value Output -> VCC; footprint (none) -> Connector_PinSocket_2.54mm:PinSocket_1x02_P2.54mm_Vertical
- Q6, Q7: footprint (none) -> Package_TO_SOT_THT:TO-5-3
- R1, R10, R11, R12, R13, R14, R15, R16, R17, R18, R19, R2, R20, R21, R22, R23, R24, R3, R4, R5, R6, R7, R8, R9: footprint (none) -> Resistor_THT:R_Axial_DIN0414_L11.9mm_D4.5mm_P15.24mm_Horizontal
- R25, R26: footprint (none) -> Resistor_THT:R_Axial_DIN0614_L14.3mm_D5.7mm_P15.24mm_Horizontal

Commit message: Add PCB
Parts:
- RV1, RV2, RV3, RV4, RV5: footprint Connector_PinSocket_2.54mm:PinSocket_1x02_P2.54mm_Vertical -> Connector_PinSocket_2.54mm:PinSocket_1x03_P2.54mm_Vertical
Other:
- note added: "Высокие"
- note added: "Низкие"
- note added: "Усиление"
Changed lines of the file:
@@
 F 0 "RV1" H 3131 2596 50  0000 R CNN
 F 1 "51K" H 3131 2505 50  0000 R CNN
-F 2 "Connector_PinSocket_2.54mm:PinSocket_1x02_P2.54mm_Vertical" H 3200 2550 50  0001 C CNN
+F 2 "Connector_PinSocket_2.54mm:PinSocket_1x03_P2.54mm_Vertical" H 3200 2550 50  0001 C CNN
 F 3 "~" H 3200 2550 50  0001 C CNN
 	1    3200 2550
@@
 F 0 "RV2" H 3581 3246 50  0000 R CNN
 F 1 "150K" H 3581 3155 50  0000 R CNN
-F 2 "Connector_PinSocket_2.54mm:PinSocket_1x02_P2.54mm_Vertical" H 3650 3200 50  0001 C CNN
+F 2 "Connector_PinSocket_2.54mm:PinSocket_1x03_P2.54mm_Vertical" H 3650 3200 50  0001 C CNN
 F 3 "~" H 3650 3200 50  0001 C CNN
 	1    3650 3200
@@
 F 0 "RV3" H 5080 3346 50  0000 R CNN
 F 1 "150K" H 5080 3255 50  0000 R CNN
-F 2 "Connector_PinSocket_2.54mm:PinSocket_1x02_P2.54mm_Vertical" H 5150 3300 50  0001 C CNN
+F 2 "Connector_PinSocket_2.54mm:PinSocket_1x03_P2.54mm_Vertical" H 5150 3300 50  0001 C CNN
 F 3 "~" H 5150 3300 50  0001 C CNN
 	1    5150 3300
@@
 F 0 "RV4" H 6080 1346 50  0000 R CNN
 F 1 "47K" H 6080 1255 50  0000 R CNN
-F 2 "Connector_PinSocket_2.54mm:PinSocket_1x02_P2.54mm_Vertical" H 6150 1300 50  0001 C CNN
+F 2 "Connector_PinSocket_2.54mm:PinSocket_1x03_P2.54mm_Vertical" H 6150 1300 50  0001 C CNN
 F 3 "~" H 6150 1300 50  0001 C CNN
 	1    6150 1300
@@
 F 0 "RV5" H 7930 3046 50  0000 R CNN
 F 1 "2K2" H 7930 2955 50  0000 R CNN
-F 2 "Connector_PinSocket_2.54mm:PinSocket_1x02_P2.54mm_Vertical" H 8000 3000 50  0001 C CNN
+F 2 "Connector_PinSocket_2.54mm:PinSocket_1x03_P2.54mm_Vertical" H 8000 3000 50  0001 C CNN
 F 3 "~" H 8000 3000 50  0001 C CNN
 	1    8000 3000
@@
 Text Label 10000 1000 0    50   ~ 0
 -20V
+Text Notes 3250 2400 0    50   ~ 0
+Усиление
+Text Notes 3250 3050 0    50   ~ 0
+Низкие
+Text Notes 5200 3150 0    50   ~ 0
+Высокие
 $EndSCHEMATC

Commit message: Fix power nets
Parts:
- removed J3: VCC, Connector_PinSocket_2.54mm:PinSocket_1x02_P2.54mm_Vertical, symbol Connector_Generic:Conn_01x02
Changed lines of the file:
@@
-	1    0    0    -1
-$EndComp
-$Comp
-L Connector_Generic:Conn_01x02 J3
-U 1 1 5E7CDEC1
-P 10400 1000
-F 0 "J3" H 10480 992 50  0000 L CNN
-F 1 "VCC" H 10480 901 50  0000 L CNN
-F 2 "Connector_PinSocket_2.54mm:PinSocket_1x02_P2.54mm_Vertical" H 10400 1000 50  0001 C CNN
-F 3 "~" H 10400 1000 50  0001 C CNN
-	1    10400 1000
-	1    0    0    -1
-$EndComp
-$Comp
-L power:GND #PWR0104
-U 1 1 5E7D3A29
-P 10100 1150
-F 0 "#PWR0104" H 10100 900 50  0001 C CNN
-F 1 "GND" H 10105 977 50  0000 C CNN
-F 2 "" H 10100 1150 50  0001 C CNN
-F 3 "" H 10100 1150 50  0001 C CNN
-	1    10100 1150
 	1    0    0    -1
 $EndComp
 Wire Wire Line
-	10200 1100 10100 1100
-Wire Wire Line
-	10100 1100 10100 1150
-Wire Wire Line
 	9450 1000 10200 1000
-Text Label 10000 1000 0    50   ~ 0
--20V
 Text Notes 3250 2400 0    50   ~ 0
 Усиление
@@
 Text Notes 5200 3150 0    50   ~ 0
 Высокие
+$Comp
+L components:-20V #PWR0102
+U 1 1 60A9364B
+P 10200 900
+F 0 "#PWR0102" H 10200 1000 50  0001 C CNN
+F 1 "-20V" H 10215 1073 50  0000 C CNN
+F 2 "" H 10200 900 50  0001 C CNN
+F 3 "" H 10200 900 50  0001 C CNN
+	1    10200 900
+	1    0    0    -1
+$EndComp
+Wire Wire Line
+	10200 1000 10200 900
+$Comp
+L power:PWR_FLAG #FLG0101
+U 1 1 60A99ED9
+P 950 900
+F 0 "#FLG0101" H 950 975 50  0001 C CNN
+F 1 "PWR_FLAG" H 950 1073 50  0000 C CNN
+F 2 "" H 950 900 50  0001 C CNN
+F 3 "~" H 950 900 50  0001 C CNN
+	1    950  900
+	-1   0    0    1
+$EndComp
+$Comp
+L components:-20V #PWR0104
+U 1 1 60A9AA08
+P 950 750
+F 0 "#PWR0104" H 950 850 50  0001 C CNN
+F 1 "-20V" H 965 923 50  0000 C CNN
+F 2 "" H 950 750 50  0001 C CNN
+F 3 "" H 950 750 50  0001 C CNN
+	1    950  750
+	1    0    0    -1
+$EndComp
+Wire Wire Line
+	950  750  950  900
+$Comp
+L power:GND #PWR0105
+U 1 1 60AA6565
+P 1350 900
+F 0 "#PWR0105" H 1350 650 50  0001 C CNN
+F 1 "GND" H 1355 727 50  0000 C CNN
+F 2 "" H 1350 900 50  0001 C CNN
+F 3 "" H 1350 900 50  0001 C CNN
+	1    1350 900
+	1    0    0    -1
+$EndComp
+$Comp
+L power:PWR_FLAG #FLG0102
+U 1 1 60AA6FD3
+P 1350 750
+F 0 "#FLG0102" H 1350 825 50  0001 C CNN
+F 1 "PWR_FLAG" H 1350 923 50  0000 C CNN
+F 2 "" H 1350 750 50  0001 C CNN
+F 3 "~" H 1350 750 50  0001 C CNN
+	1    1350 750
+	1    0    0    -1
+$EndComp
+Wire Wire Line
+	1350 750  1350 900
 $EndSCHEMATC

Commit message: Add preamp schematic
Parts:
- added C1: 5u x 15V, Capacitor_THT:CP_Radial_D4.0mm_P2.00mm, symbol Device:CP
- added C2, C5: 15u x 6V, Capacitor_THT:CP_Radial_D5.0mm_P2.00mm, symbol Device:CP
- added C3: 120p, Capacitor_THT:C_Rect_L4.6mm_W3.8mm_P2.50mm_MKS02_FKP02, symbol Device:C
- added C4: 5u x 10V, Capacitor_THT:CP_Radial_D4.0mm_P2.00mm, symbol Device:CP
- added C6: 33u x 20V, Capacitor_THT:CP_Radial_D5.0mm_P2.00mm, symbol Device:CP
- added D1: Д813, symbol Device:D
- added J1: Input, Connector_PinSocket_2.54mm:PinSocket_1x02_P2.54mm_Vertical, symbol Connector_Generic:Conn_01x02
- added J2: Output, Connector_PinSocket_2.54mm:PinSocket_1x02_P2.54mm_Vertical, symbol Connector_Generic:Conn_01x02
- added Q1, Q2: П28, Package_TO_SOT_THT:TO-11-3, symbol Device:Q_PNP_BEC
- added R1: 6.8K, symbol Device:R
- added R10, R8: 1K, symbol Device:R
- added R2: 150, symbol Device:R
- added R3: 3K, symbol Device:R
- added R4: 75K, symbol Device:R
- added R5: 120K, symbol Device:R
- added R6: 8.2K, symbol Device:R
- added R7: 1.2K, symbol Device:R
- added R9: 590, symbol Device:R
- C11: renamed from C5; value 22n -> 0.022u
- C12: renamed from C6; value 100n -> 0.22u
- C13: renamed from C7; value 10n -> 0.1u
- C14: renamed from C8; value 100n -> 0.01u
- renumbered C4 to C10, C9 to C15, C10 to C16, C11 to C17, C12 to C18, C13 to C19, C14 to C20, C1 to C7, C2 to C8, C3 to C9, J1 to J3, J2 to J4, Q1 to Q3, Q2 to Q4, Q3 to Q5, Q4 to Q6, Q5 to Q7, Q6 to Q8, Q7 to Q9, R1 to R11, R2 to R12, R3 to R13, R4 to R14, R5 to R15, R6 to R16, R7 to R17, R8 to R18, R9 to R19, R10 to R20, R11 to R21, R12 to R22, R13 to R23, R14 to R24, R15 to R25, R16 to R26, R17 to R27, R18 to R28, R19 to R29, R20 to R30, R21 to R31, R22 to R32, R23 to R33, R24 to R34, R25 to R35, R26 to R36
Connections:
- net -20V: now also R10.1
- net GND: now also C2.1, C6.1, D1.1 (K), J1.2 (Pin_2), J2.2 (Pin_2), R3.2, R8.2, R9.2
- new net: C1.1, J1.1 (Pin_1)
- new net: C1.2, Q1.1 (B), R1.1
- new net: C3.2, Q1.2 (E), R2.1, R4.2
- new net: Q1.3 (C), Q2.1 (B), R5.2
- new net: R1.2, R7.2, R8.1
- new net: C2.2, R2.2, R3.1
- new net: C3.1, R4.1
- new net: C5.2, Q2.2 (E), R7.1
- new net: C4.2, Q2.3 (C), R6.2
- new net: C6.2, D1.2 (A), R10.2, R5.1, R6.1
- new net: C4.1, J2.1 (Pin_1)
- new net: C5.1, R9.1
Other:
- moved on the sheet: C10, C11, C12, C13, C14, C15, C16, C17, C18, C19, C20, C7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

Commit message: Assign footprints to components
Parts:
- C10: footprint Capacitor_THT:CP_Radial_D10.0mm_P5.00mm -> Capacitor_THT:CP_Radial_D5.0mm_P2.00mm
- C12: footprint Capacitor_THT:C_Rect_L11.0mm_W3.4mm_P10.00mm_MKT -> Capacitor_THT:C_Disc_D14.5mm_W5.0mm_P7.50mm
- C13: footprint Capacitor_THT:C_Disc_D4.7mm_W2.5mm_P5.00mm -> Capacitor_THT:C_Disc_D14.5mm_W5.0mm_P7.50mm
- C14: footprint Capacitor_THT:C_Rect_L11.0mm_W3.4mm_P10.00mm_MKT -> Capacitor_THT:C_Disc_D7.5mm_W4.4mm_P5.00mm
- C15, C9: footprint Capacitor_THT:CP_Radial_D7.5mm_P2.50mm -> Capacitor_THT:CP_Radial_D4.0mm_P2.00mm
- C16: footprint Capacitor_THT:CP_Radial_D12.5mm_P5.00mm -> Capacitor_THT:CP_Radial_D8.0mm_P3.50mm
- C17, C19, C20: footprint Capacitor_THT:CP_Radial_D8.0mm_P3.50mm -> Capacitor_THT:CP_Radial_D5.0mm_P2.00mm
- C18: value 1n -> 0.001u; footprint Capacitor_THT:C_Disc_D4.7mm_W2.5mm_P5.00mm -> Capacitor_THT:C_Rect_L4.6mm_W3.8mm_P2.50mm_MKS02_FKP02
- D1: footprint (none) -> Diode_THT:D_DO-201_P15.24mm_Horizontal
- R1, R10, R2, R3, R4, R5, R6, R7, R8, R9: footprint (none) -> Resistor_THT:R_Axial_DIN0309_L9.0mm_D3.2mm_P12.70mm_Horizontal
- R11, R12, R13, R14, R15, R16, R18, R19, R20, R21, R22, R23, R24, R25, R26, R27, R28, R29, R31, R33, R34: footprint Resistor_THT:R_Axial_DIN0414_L11.9mm_D4.5mm_P15.24mm_Horizontal -> Resistor_THT:R_Axial_DIN0309_L9.0mm_D3.2mm_P12.70mm_Horizontal
- R17: value 6K2 -> 6.2K; footprint Resistor_THT:R_Axial_DIN0414_L11.9mm_D4.5mm_P15.24mm_Horizontal -> Resistor_THT:R_Axial_DIN0309_L9.0mm_D3.2mm_P12.70mm_Horizontal
- R30: value 2K4 -> 2.4K; footprint Resistor_THT:R_Axial_DIN0414_L11.9mm_D4.5mm_P15.24mm_Horizontal -> Resistor_THT:R_Axial_DIN0309_L9.0mm_D3.2mm_P12.70mm_Horizontal
- R32: value 1K8 -> 1.8K; footprint Resistor_THT:R_Axial_DIN0414_L11.9mm_D4.5mm_P15.24mm_Horizontal -> Resistor_THT:R_Axial_DIN0309_L9.0mm_D3.2mm_P12.70mm_Horizontal
- R35, R36: footprint Resistor_THT:R_Axial_DIN0614_L14.3mm_D5.7mm_P15.24mm_Horizontal -> Resistor_THT:R_Axial_DIN0918_L18.0mm_D9.0mm_P25.40mm_Horizontal
- RV5: value 2K2 -> 2.2K

Commit message: Route preamp
Parts:
- added J5: Power, Connector_PinSocket_2.54mm:PinSocket_1x02_P2.54mm_Vertical, symbol Connector_Generic:Conn_01x02
Connections:
- net -20V: now also J5.1 (Pin_1)
- net GND: now also J5.2 (Pin_2)
- net at C3.1, R4.1: now also C4.2, Q2.3 (C), R6.2
Other:
- moved on the sheet: R5
Changed lines of the file:
@@
 	2450 2500 2450 2400
 Wire Wire Line
-	2450 2400 3300 2400
-Wire Wire Line
-	3300 2400 3300 2750
-Wire Wire Line
-	3300 2750 3400 2750
+	2450 2400 3100 2400
+Wire Wire Line
+	3100 2400 3100 2750
+Wire Wire Line
+	3100 2750 3400 2750
 $Comp
 L Device:R R5
 U 1 1 60BCF1E0
-P 3300 2050
-F 0 "R5" H 3370 2096 50  0000 L CNN
-F 1 "120K" H 3370 2005 50  0000 L CNN
-F 2 "Resistor_THT:R_Axial_DIN0309_L9.0mm_D3.2mm_P12.70mm_Horizontal" V 3230 2050 50  0001 C CNN
-F 3 "~" H 3300 2050 50  0001 C CNN
-	1    3300 2050
-	1    0    0    -1
-$EndComp
-Wire Wire Line
-	3300 2200 3300 2400
-Connection ~ 3300 2400
+P 3100 2050
+F 0 "R5" H 3170 2096 50  0000 L CNN
+F 1 "120K" H 3170 2005 50  0000 L CNN
+F 2 "Resistor_THT:R_Axial_DIN0309_L9.0mm_D3.2mm_P12.70mm_Horizontal" V 3030 2050 50  0001 C CNN
+F 3 "~" H 3100 2050 50  0001 C CNN
+	1    3100 2050
+	1    0    0    -1
+$EndComp
+Connection ~ 3100 2400
 $Comp
 L Device:R R6
@@
 $EndComp
 Wire Wire Line
-	3300 1850 3300 1900
+	3100 1850 3100 1900
 Wire Wire Line
 	3700 1900 3700 1850
 Connection ~ 3700 1850
 Wire Wire Line
-	3700 1850 3300 1850
+	3700 1850 3100 1850
 Wire Wire Line
 	3700 1850 4550 1850
@@
 Wire Wire Line
 	5100 1850 4950 1850
+Wire Wire Line
+	3250 3000 3350 3000
+Wire Wire Line
+	3350 3000 3350 2400
+Wire Wire Line
+	3350 2400 3700 2400
+Connection ~ 3250 3000
+Wire Wire Line
+	3100 2200 3100 2400
+$Comp
+L Connector_Generic:Conn_01x02 J5
+U 1 1 60BDE341
+P 1650 1000
+F 0 "J5" H 1568 1217 50  0000 C CNN
+F 1 "Power" H 1568 1126 50  0000 C CNN
+F 2 "Connector_PinSocket_2.54mm:PinSocket_1x02_P2.54mm_Vertical" H 1650 1000 50  0001 C CNN
+F 3 "~" H 1650 1000 50  0001 C CNN
+	1    1650 1000
+	-1   0    0    -1
+$EndComp
+$Comp
+L components:-20V #PWR010
+U 1 1 60BDEDE6
+P 2050 950
+F 0 "#PWR010" H 2050 1050 50  0001 C CNN
+F 1 "-20V" H 2065 1123 50  0000 C CNN
+F 2 "" H 2050 950 50  0001 C CNN
+F 3 "" H 2050 950 50  0001 C CNN
+	1    2050 950
+	1    0    0    -1
+$EndComp
+Wire Wire Line
+	2050 950  2050 1000
+Wire Wire Line
+	2050 1000 1850 1000
+$Comp
+L power:GND #PWR011
+U 1 1 60BEEEA5
+P 2050 1200
+F 0 "#PWR011" H 2050 950 50  0001 C CNN
+F 1 "GND" H 2055 1027 50  0000 C CNN
+F 2 "" H 2050 1200 50  0001 C CNN
+F 3 "" H 2050 1200 50  0001 C CNN
+	1    2050 1200
+	1    0    0    -1
+$EndComp
+Wire Wire Line
+	2050 1200 2050 1100
+Wire Wire Line
+	2050 1100 1850 1100
 $EndSCHEMATC
